File: v2/ab.brd (EAGLE design)
At the start: 26 x 22.7 mm, 5 parts

Commit message: Update to v2.1
Parts:
- TP0, TP1: value TPPAD1-13 -> TESTPAD; device testpad:P1-13 -> lib:TESTPAD
Connections:
- net N$1: now also TP0.P$1; no longer TP0.TP
- net N$3: now also TP1.P$1; no longer TP1.TP
Routing:
- net N$2: track 0.00 -> 85.5 mm
- net GND: track 6.90 -> 8.60 mm
Other:
- board size 26 x 22.7 mm -> 26 x 21.7 mm
- board text added: "AGB_TACT_ab_V2.1"
- board text removed: "AGB_TACT_ab_V2.0"
