File: v2/ab.sch (EAGLE design)
At the start: 5 parts

Commit message: Update to v2.1
Parts:
- TP0, TP1: value TPPAD1-13 -> TESTPAD; device testpad:TPPAD1-13 -> lib:TESTPAD
Changed lines of the file:
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@@
 </classes>
 <parts>
-<part name="TP0" library="testpad" library_urn="urn:adsk.eagle:library:385" deviceset="TP" device="PAD1-13" package3d_urn="urn:adsk.eagle:package:27946/1"/>
-<part name="TP1" library="testpad" library_urn="urn:adsk.eagle:library:385" deviceset="TP" device="PAD1-13" package3d_urn="urn:adsk.eagle:package:27946/1"/>
+<part name="TP0" library="lib" deviceset="TESTPAD" device="">
+<attribute name="TP_SIGNAL_NAME" value=""/>
+</part>
+<part name="TP1" library="lib" deviceset="TESTPAD" device="">
+<attribute name="TP_SIGNAL_NAME" value=""/>
+</part>
 <part name="GND" library="testpad" library_urn="urn:adsk.eagle:library:385" deviceset="TP" device="PAD1-13" package3d_urn="urn:adsk.eagle:package:27946/1"/>
 <part name="SUPPLY1" library="supply2" library_urn="urn:adsk.eagle:library:372" deviceset="GND" device=""/>
